File: hardware/Jetson_USB.kicad_sch (KiCad schematic)
At the start: 15 parts, among them J5 USB_B_Mini, U3 USBLC6-2SC6, U6 FT230XS

Commit message: JLC assembly parts
Parts:
- C10: JLC (none) -> C1779
- C12, C15, C17: JLC (none) -> C49678
- D12, D13: JLC (none) -> C84256
- J5: MPN (none) -> MUSB-B5-S-VT-02; now left out of the parts list
- R18, R19: MPN (none) -> RC0805JR-0727RL; now left out of the parts list
- R20, R21: value 270 -> 300; JLC (none) -> C17617
- R22: JLC (none) -> C17414
- R23: JLC (none) -> C17673
- U3: JLC (none) -> C2827654
- U6: JLC (none) -> C69082
Changed lines of the file:
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@@
 		(unit 1)
 		(exclude_from_sim no)
-		(in_bom yes)
+		(in_bom no)
 		(on_board yes)
 		(dnp no)
@@
 			)
 		)
+		(property "MPN" "MUSB-B5-S-VT-02"
+			(at 58.42 88.9 0)
+			(effects
+				(font
+					(size 1.27 1.27)
+				)
+				(hide yes)
+			)
+		)
 		(pin "2"
 		)
@@
 			)
 		)
+		(property "JLC" "C1779"
+			(at 193.04 66.04 0)
+			(effects
+				(font
+					(size 1.27 1.27)
+				)
+				(hide yes)
+			)
+		)
 		(pin "1"
 		)
@@
 			)
 		)
+		(property "JLC" "C49678"
+			(at 118.11 100.33 0)
+			(effects
+				(font
+					(size 1.27 1.27)
+				)
+				(hide yes)
+			)
+		)
 		(pin "1"
 		)
@@
 		)
 		(property "Description" ""
+			(at 203.2 66.04 0)
+			(effects
+				(font
+					(size 1.27 1.27)
+				)
+				(hide yes)
+			)
+		)
+		(property "JLC" "C49678"
 			(at 203.2 66.04 0)
 			(effects
@@
 		(unit 1)
 		(exclude_from_sim no)
-		(in_bom yes)
+		(in_bom no)
 		(on_board yes)
 		(dnp no)
@@
 			)
 		)
+		(property "JLC" ""
+			(at 133.35 86.36 0)
+			(effects
+				(font
+					(size 1.27 1.27)
+				)
+				(hide yes)
+			)
+		)
+		(property "MPN" "RC0805JR-0727RL"
+			(at 133.35 86.36 0)
+			(effects
+				(font
+					(size 1.27 1.27)
+				)
+				(hide yes)
+			)
+		)
 		(pin "2"
 		)
@@
 		(unit 1)
 		(exclude_from_sim no)
-		(in_bom yes)
+		(in_bom no)
 		(on_board yes)
 		(dnp no)
@@
 			)
 		)
+		(property "JLC" ""
+			(at 133.35 88.9 0)
+			(effects
+				(font
+					(size 1.27 1.27)
+				)
+				(hide yes)
+			)
+		)
+		(property "MPN" "RC0805JR-0727RL"
+			(at 133.35 88.9 0)
+			(effects
+				(font
+					(size 1.27 1.27)
+				)
+				(hide yes)
+			)
+		)
 		(pin "2"
 		)
@@
 			)
 		)
+		(property "JLC" "C84256"
+			(at 184.15 106.68 0)
+			(effects
+				(font
+					(size 1.27 1.27)
+				)
+				(hide yes)
+			)
+		)
 		(pin "1"
 		)
@@
 			)
 		)
-		(property "Value" "270"
+		(property "Value" "300"
 			(at 179.07 116.84 90)
 			(effects
@@
 			)
 		)
+		(property "JLC" "C17617"
+			(at 179.07 114.3 0)
+			(effects
+				(font
+					(size 1.27 1.27)
+				)
+				(hide yes)
+			)
+		)
 		(pin "2"
 		)
@@
 			)
 		)
+		(property "JLC" "C84256"
+			(at 184.15 114.3 0)
+			(effects
+				(font
+					(size 1.27 1.27)
+				)
+				(hide yes)
+			)
+		)
 		(pin "1"
 		)
@@
 		)
 		(property "Description" ""
+			(at 214.63 66.04 0)
+			(effects
+				(font
+					(size 1.27 1.27)
+				)
+				(hide yes)
+			)
+		)
+		(property "JLC" "C49678"
 			(at 214.63 66.04 0)
 			(effects
@@
 			)
 		)
+		(property "JLC" "C2827654"
+			(at 58.42 140.97 0)
+			(effects
+				(font
+					(size 1.27 1.27)
+				)
+				(hide yes)
+			)
+		)
 		(pin "2"
 		)
@@
 			)
 		)
+		(property "JLC" "C69082"
+			(at 153.67 88.9 0)
+			(effects
+				(font
+					(size 1.27 1.27)
+				)
+				(hide yes)
+			)
+		)
 		(pin "6"
 		)
@@
 			)
 		)
+		(property "JLC" "C17414"
+			(at 184.15 93.98 0)
+			(effects
+				(font
+					(size 1.27 1.27)
+				)
+				(hide yes)
+			)
+		)
 		(pin "2"
 		)
@@
 			)
 		)
+		(property "JLC" "C17673"
+			(at 184.15 88.9 0)
+			(effects
+				(font
+					(size 1.27 1.27)
+				)
+				(hide yes)
+			)
+		)
 		(pin "2"
 		)
@@
 			)
 		)
-		(property "Value" "270"
+		(property "Value" "300"
 			(at 179.07 109.22 90)
 			(effects
@@
 			(at 179.07 106.68 0)
 			(effects
+				(font
+					(size 1.27 1.27)
+				)
+				(hide yes)
+			)
+		)
+		(property "JLC" "C17617"
+			(at 179.07 106.68 0)
+			(effects

Commit message: Schematic cleanup
Parts:
- removed J5: USB_B_Mini, AMP_Custom:USB_Mini-B_Adam_Tech_MUSB-B5-S-VT-02_Vertical_CircularHoles, symbol Connector:USB_B_Mini
Connections:
- no-connect marks 6 -> 5
Other:
- moved on the sheet: U3

Commit message: Final touches for assembly
Parts:
- U3: JLCPCB Rotation Offset (none) -> 90
Changed lines of the file:
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@@
+			)
+		)
+		(property "JLCPCB Rotation Offset" "90"
+			(at 138.43 139.7 0)
+			(effects
+				(font
+					(size 1.27 1.27)
+				)
+				(hide yes)
 			)
 		)
