File: hardware/IMU.kicad_sch (KiCad schematic)
At the start: 6 parts, among them U5 ICM-20948, U7 TLV74318P

Commit message: Add level shifter for LEDs
Parts:
- renumbered C15 to C11, C16 to C14, C14 to C16, U7 to U4
Changed lines of the file:
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@@
 		(dnp no)
 		(fields_autoplaced yes)
-		(property "Reference" "C16"
+		(property "Reference" "C14"
 			(at 161.29 102.8763 0)
 			(effects
@@
 			(project "AMP_PCBv3"
 				(path "/b0eed686-2b97-4c99-952c-ca5393e47dfe/8b192e67-3643-4fb6-9eaf-c07d80095f2d"
-					(reference "C16")
+					(reference "C14")
 					(unit 1)
 				)
@@
 		(on_board yes)
 		(dnp no)
-		(property "Reference" "C14"
+		(property "Reference" "C16"
 			(at 165.1 80.0163 0)
 			(effects
@@
 			(project "AMP_PCBv3"
 				(path "/b0eed686-2b97-4c99-952c-ca5393e47dfe/8b192e67-3643-4fb6-9eaf-c07d80095f2d"
-					(reference "C14")
+					(reference "C16")
 					(unit 1)
 				)
@@
 		(dnp no)
 		(fields_autoplaced yes)
-		(property "Reference" "U7"
+		(property "Reference" "U4"
 			(at 100.33 76.2 0)
 			(effects
@@
 			(project "AMP_PCBv3"
 				(path "/b0eed686-2b97-4c99-952c-ca5393e47dfe/8b192e67-3643-4fb6-9eaf-c07d80095f2d"
-					(reference "U7")
+					(reference "U4")
 					(unit 1)
 				)
@@
 		(dnp no)
 		(fields_autoplaced yes)
-		(property "Reference" "C15"
+		(property "Reference" "C11"
 			(at 175.26 80.0163 0)
 			(effects
@@
 			(project "AMP_PCBv3"
 				(path "/b0eed686-2b97-4c99-952c-ca5393e47dfe/8b192e67-3643-4fb6-9eaf-c07d80095f2d"
-					(reference "C15")
-					(unit 1)
-				)
+					(reference "C11")
+					(unit 1)
+				)

Commit message: JLC assembly parts
Parts:
- C11, C14, C16: JLC (none) -> C49678
- C13: JLC (none) -> C28323
- U4: JLC (none) -> C485152
- U5: JLC (none) -> C726001
Changed lines of the file:
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@@
+			)
+		)
+		(property "JLC" "C28323"
+			(at 110.49 85.09 0)
+			(effects
+				(font
+					(size 1.27 1.27)
+				)
+				(hide yes)
 			)
 		)
@@
 			)
 		)
+		(property "JLC" "C49678"
+			(at 158.75 104.14 0)
+			(effects
+				(font
+					(size 1.27 1.27)
+				)
+				(hide yes)
+			)
+		)
 		(pin "1"
 		)
@@
 			)
 		)
+		(property "JLC" "C49678"
+			(at 167.64 81.28 0)
+			(effects
+				(font
+					(size 1.27 1.27)
+				)
+				(hide yes)
+			)
+		)
 		(pin "1"
 		)
@@
 			)
 		)
+		(property "JLC" "C726001"
+			(at 143.51 96.52 0)
+			(effects
+				(font
+					(size 1.27 1.27)
+				)
+				(hide yes)
+			)
+		)
 		(pin "7"
 		)
@@
 			)
 		)
+		(property "JLC" "C485152"
+			(at 100.33 85.09 0)
+			(effects
+				(font
+					(size 1.27 1.27)
+				)
+				(hide yes)
+			)
+		)
 		(pin "1"
 		)
@@
 			(at 172.72 81.28 0)
 			(effects
+				(font
+					(size 1.27 1.27)
+				)
+				(hide yes)
+			)
+		)
+		(property "JLC" "C49678"
+			(at 172.72 81.28 0)
+			(effects

Commit message: Schematic cleanup
Connections:
- net CS renamed NSS
Other:
- note added: "1.8V REGULATOR"
- note added: "IMU"
- title: IMU -> AMP PCBv3
- moved on the sheet: C11, C13, C14, C16, U4, U5

Commit message: Final touches for assembly
Parts:
- U5: JLCPCB Rotation Offset (none) -> -90
Changed lines of the file:
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@@
+			)
+		)
+		(property "JLCPCB Rotation Offset" "-90"
+			(at 151.13 96.52 0)
+			(effects
+				(font
+					(size 1.27 1.27)
+				)
+				(hide yes)
 			)
 		)
